Commit message: Revert "Humble development"

File: uuv_sensor_plugins/uuv_sensor_ros_plugins/urdf/dvl_snippets.xacro (robot description, xacro)
@@ -44,5 +44,5 @@
       namespace="${namespace}"
       parent_link="${parent_link}"
-      inertial_reference_frame="world">
+      reference_frame="world">
       <xacro:insert_block name="origin" />
     </xacro:default_dvl_macro>
@@ -52,5 +52,5 @@
       namespace="${namespace}"
       parent_link="${parent_link}"
-      inertial_reference_frame="world_ned">
+      reference_frame="world_ned">
       <xacro:insert_block name="origin" />
     </xacro:default_dvl_macro>
@@ -71,5 +71,5 @@
     </xacro:dvl_plugin_macro>
   </xacro:macro>
-  <xacro:macro name="dvl_single_sonar" params="namespace suffix index pitch yaw update_rate topic">
+  <xacro:macro name="dvl_single_sonar" params="namespace suffix index pitch yaw update_rate">
     <link name="${namespace}/dvl${suffix}_sonar${index}_link">
       <inertial>
@@ -120,5 +120,4 @@
         <plugin filename="libgazebo_ros_ray_sensor.so" name="dvl${suffix}_sonar${index}">
           <ros>
-            <namespace>${namespace}</namespace>
             <remapping>~/out:=${topic}_sonar${index}</remapping>
           </ros>
@@ -162,17 +161,17 @@
     <xacro:dvl_single_sonar
       namespace="${namespace}" suffix=""
-      index="0" pitch="-0.52" yaw="0.0" update_rate="${update_rate}" topic="${topic}">
-    </xacro:dvl_single_sonar>
-    <xacro:dvl_single_sonar
-      namespace="${namespace}" suffix=""
-      index="1" pitch="0" yaw="0.52" update_rate="${update_rate}" topic="${topic}">
-    </xacro:dvl_single_sonar>
-    <xacro:dvl_single_sonar
-      namespace="${namespace}" suffix=""
-      index="2" pitch="0.52" yaw="0.0" update_rate="${update_rate}" topic="${topic}">
-    </xacro:dvl_single_sonar>
-    <xacro:dvl_single_sonar
-      namespace="${namespace}" suffix=""
-      index="3" pitch="0.0" yaw="-0.52" update_rate="${update_rate}" topic="${topic}">
+      index="0" pitch="-0.52" yaw="0.0" update_rate="${update_rate}">
+    </xacro:dvl_single_sonar>
+    <xacro:dvl_single_sonar
+      namespace="${namespace}" suffix=""
+      index="1" pitch="0" yaw="0.52" update_rate="${update_rate}">
+    </xacro:dvl_single_sonar>
+    <xacro:dvl_single_sonar
+      namespace="${namespace}" suffix=""
+      index="2" pitch="0.52" yaw="0.0" update_rate="${update_rate}">
+    </xacro:dvl_single_sonar>
+    <xacro:dvl_single_sonar
+      namespace="${namespace}" suffix=""
+      index="3" pitch="0.0" yaw="-0.52" update_rate="${update_rate}">
     </xacro:dvl_single_sonar>
     <gazebo>

File: uuv_sensor_plugins/uuv_sensor_ros_plugins/urdf/sonar_snippets.xacro (robot description, xacro)
@@ -145,6 +145,5 @@
         </noise>
       </ray>
-      <plugin name="sonar${suffix}_controller" filename="libgazebo_ros_ray_sensor.so">
-        <namespace>${namespace}</namespace>
+      <plugin name="sonar${suffix}_controller" filename="libgazebo_ros_gpu_laser.so">
         <topicName>${topic}</topicName>
         <frameName>sonar${suffix}_link</frameName>
